Commit message: created lidar plugin

File: description/lidar_plugin.xacro (robot description, xacro)
@@ -1,32 +1,25 @@
 <?xml version="1.0"?>
-<robot xmlns:xacro="http://www.ros.org/wiki/xacro">
-    <xacro:include filename="inertial_macros.xacro" />
-    <joint name="lidar_joint" type="fixed">
-        <origin xyz="0.2 0.0 0.09" rpy="0.0 0.0 0.0"/>
-        <parent link="chassis_link"/>
-        <child link="lidar_link"/>
-        <axis xyz="0.0 0.0 0.0"/>
-    </joint>
-    <link name="lidar_link">
-        <visual>
-            <origin xyz="0.0 0.0 0.0" rpy="0.0 0.0 0.0"/>
-            <geometry>
-                <cylinder radius="0.035" length="0.02"/>
-            </geometry>
-            <material name="black">
-                <color rgba="0.0 0.0 0.0 1.0"/>
-            </material>
-        </visual>
-        <collision>
-            <geometry>
-                <cylinder radius="0.035" length="0.02"/>
-            </geometry>
-        </collision>
-        <xacro:inertial_cylinder mass="0.1" radius="0.035" length="0.02">
-             <origin xyz="0 0 0" rpy=" 0 0 0"/>
-        </xacro:inertial_cylinder>
-    </link>
-    <!--laser plugin-->
-    <gazebo reference="lidar_link">
+<robot xmlns:xacro="http://www.ros.org/wiki/xacro" >
+<joint name="lidar_joint" type="fixed">
+    <origin xyz="0.0 0.0 0.0" rpy="0.0 0.0 0.0"/>
+    <parent link="chassis_link"/>
+    <child link="lidar_link"/>
+    <axis xyz="0.0 0.0 0.0"/>
+</joint>
+<link name="lidar_link">
+    <visual>
+        <origin xyz="0.0 0.0 0.0" rpy="0.0 0.0 0.0"/>
+        <geometry>
+            <cylinder radius="0.07" length="0.05"/>
+        </geometry>
+        <material name="black"/>
+    </visual>
+    <collision>
+        <geometry>
+            <cylinder radius="0.07" length="0.05"/>
+        </geometry>
+    </collision>
+</link>
+<gazebo reference="lidar_link">
         <material>Gazebo/White</material>
         <sensor name="lidar" type="ray">
@@ -47,5 +40,5 @@
                 </range>
             </ray>
-            <plugin name="laser_controller" filename="libgazebo_ros_ray_sensor.so">
+            <plugin name="lidar_controller" filename="libgazebo_ros_ray_sensor.so">
                 <ros>
                     <argument>~/out:=scan</argument>

File: description/robot_core.xacro (robot description, xacro)
@@ -16,4 +16,13 @@
 <!--BASE_LINK-->
     <link name="base_link">
+    </link>
+<!--Base_footprint-->
+    <joint name="base_footprint_joint" type="fixed">
+        <origin xyz="0.0 0.0 0.0" rpy="0.0 0.0 0.0"/>
+        <parent link="base_link"/>
+        <child link="base_link"/>
+        <axis xyz="0.0 0.0 0.0"/>
+    </joint>
+    <link name="base_footprint">
     </link>
 <!--CHASSIS_LINK-->

Commit message: created lidar plugin in urdf

File: description/lidar_plugin.xacro (robot description, xacro)
@@ -9,5 +9,5 @@
 <link name="lidar_link">
     <visual>
-        <origin xyz="0.0 0.0 0.0" rpy="0.0 0.0 0.0"/>
+        <origin xyz="0.0 0.0 0.08 " rpy="0.0 0.0 0.0"/>
         <geometry>
             <cylinder radius="0.07" length="0.05"/>

File: description/robot_core.xacro (robot description, xacro)
@@ -21,5 +21,5 @@
         <origin xyz="0.0 0.0 0.0" rpy="0.0 0.0 0.0"/>
         <parent link="base_link"/>
-        <child link="base_link"/>
+        <child link="base_footprint"/>
         <axis xyz="0.0 0.0 0.0"/>
     </joint>

Commit message: created lidar_plugin

File: description/lidar_plugin.xacro (robot description, xacro)
@@ -2,5 +2,5 @@
 <robot xmlns:xacro="http://www.ros.org/wiki/xacro" >
 <joint name="lidar_joint" type="fixed">
-    <origin xyz="0.0 0.0 0.0" rpy="0.0 0.0 0.0"/>
+    <origin xyz="0.1 0.0 0.04" rpy="0.0 0.0 0.0"/>
     <parent link="chassis_link"/>
     <child link="lidar_link"/>
@@ -9,7 +9,7 @@
 <link name="lidar_link">
     <visual>
-        <origin xyz="0.0 0.0 0.08 " rpy="0.0 0.0 0.0"/>
+        <origin xyz="0.1 0.0 0.04 " rpy="0.0 0.0 0.0"/>
         <geometry>
-            <cylinder radius="0.07" length="0.05"/>
+            <cylinder radius="0.035" length="0.05"/>
         </geometry>
         <material name="black"/>
@@ -17,5 +17,5 @@
     <collision>
         <geometry>
-            <cylinder radius="0.07" length="0.05"/>
+            <cylinder radius="0.035" length="0.05"/>
         </geometry>
     </collision>
@@ -25,5 +25,5 @@
         <sensor name="lidar" type="ray">
             <pose> 0 0 0 0 0 0 </pose>
-            <visualize>false</visualize>
+            <visualize>true</visualize>
             <update_rate>10</update_rate>
             <ray>

Commit message: changed_urdf

File: description/lidar_plugin.xacro (robot description, xacro)
@@ -1,24 +1,4 @@
 <?xml version="1.0"?>
 <robot xmlns:xacro="http://www.ros.org/wiki/xacro" >
-<joint name="lidar_joint" type="fixed">
-    <origin xyz="0.1 0.0 0.04" rpy="0.0 0.0 0.0"/>
-    <parent link="chassis_link"/>
-    <child link="lidar_link"/>
-    <axis xyz="0.0 0.0 0.0"/>
-</joint>
-<link name="lidar_link">
-    <visual>
-        <origin xyz="0.1 0.0 0.04 " rpy="0.0 0.0 0.0"/>
-        <geometry>
-            <cylinder radius="0.035" length="0.05"/>
-        </geometry>
-        <material name="black"/>
-    </visual>
-    <collision>
-        <geometry>
-            <cylinder radius="0.035" length="0.05"/>
-        </geometry>
-    </collision>
-</link>
 <gazebo reference="lidar_link">
         <material>Gazebo/White</material>

File: description/robot.urdf.xacro (robot description, xacro)
@@ -1,5 +1,5 @@
 <?xml version="1.0"?>
 <robot xmlns:xacro="http://www.ros.org/wiki/xacro"  name="robot">
-    <xacro:include filename="robot_core.xacro" />
+    <xacro:include filename="medox_robot.xacro" />
     <!-- <xacro:include filename="diff_drive_controller_plugin.xacro" /> -->
     <xacro:include filename="ros2_control.xacro" />

File: description/ros2_control.xacro (robot description, xacro)
@@ -49,5 +49,5 @@
                 <state_interface name="position"/>
             </joint>
-    </ros2_control> -->
+    </ros2_control>-->
     <gazebo>
         <plugin name="gazebo_ros2_control" filename="libgazebo_ros2_control.so">

Commit message: original_repo

File: description/lidar_plugin.xacro (robot description, xacro)
@@ -1,4 +1,24 @@
 <?xml version="1.0"?>
 <robot xmlns:xacro="http://www.ros.org/wiki/xacro" >
+<joint name="lidar_joint" type="fixed">
+    <origin xyz="0.1 0.0 0.04" rpy="0.0 0.0 0.0"/>
+    <parent link="chassis_link"/>
+    <child link="lidar_link"/>
+    <axis xyz="0.0 0.0 0.0"/>
+</joint>
+<link name="lidar_link">
+    <visual>
+        <origin xyz="0.1 0.0 0.04 " rpy="0.0 0.0 0.0"/>
+        <geometry>
+            <cylinder radius="0.035" length="0.05"/>
+        </geometry>
+        <material name="black"/>
+    </visual>
+    <collision>
+        <geometry>
+            <cylinder radius="0.035" length="0.05"/>
+        </geometry>
+    </collision>
+</link>
 <gazebo reference="lidar_link">
         <material>Gazebo/White</material>

File: description/robot.urdf.xacro (robot description, xacro)
@@ -1,5 +1,5 @@
 <?xml version="1.0"?>
 <robot xmlns:xacro="http://www.ros.org/wiki/xacro"  name="robot">
-    <xacro:include filename="medox_robot.xacro" />
+    <xacro:include filename="robot_core.xacro" />
     <!-- <xacro:include filename="diff_drive_controller_plugin.xacro" /> -->
     <xacro:include filename="ros2_control.xacro" />

File: description/ros2_control.xacro (robot description, xacro)
@@ -49,5 +49,5 @@
                 <state_interface name="position"/>
             </joint>
-    </ros2_control>-->
+    </ros2_control> -->
     <gazebo>
         <plugin name="gazebo_ros2_control" filename="libgazebo_ros2_control.so">

Commit message: created_core_urdf

File: description/lidar_plugin.xacro (robot description, xacro)
@@ -1,24 +1,4 @@
 <?xml version="1.0"?>
 <robot xmlns:xacro="http://www.ros.org/wiki/xacro" >
-<joint name="lidar_joint" type="fixed">
-    <origin xyz="0.1 0.0 0.04" rpy="0.0 0.0 0.0"/>
-    <parent link="chassis_link"/>
-    <child link="lidar_link"/>
-    <axis xyz="0.0 0.0 0.0"/>
-</joint>
-<link name="lidar_link">
-    <visual>
-        <origin xyz="0.1 0.0 0.04 " rpy="0.0 0.0 0.0"/>
-        <geometry>
-            <cylinder radius="0.035" length="0.05"/>
-        </geometry>
-        <material name="black"/>
-    </visual>
-    <collision>
-        <geometry>
-            <cylinder radius="0.035" length="0.05"/>
-        </geometry>
-    </collision>
-</link>
 <gazebo reference="lidar_link">
         <material>Gazebo/White</material>

File: description/robot_core.xacro (robot description, xacro)
@@ -2,9 +2,7 @@
  <!--Declaration of xacro file format-->
 <robot xmlns:xacro="https://www.ros.org/wiki/xacro">
-<!--including the inertial macros file -->
-    <xacro:include filename="inertial_macros.xacro"/>
 <!--Delcaration of colors which has been used for the links-->
-    <material name="gold">
-        <color rgba="1.0 0.8 0.0 1.0"/>
+    <material name="white">
+        <color rgba="1.0 1.0 1.0 1.0"/>
     </material>
     <material name="black">
@@ -14,121 +12,401 @@
         <color rgba="1.0 0.0 0.0 1.0"/>
     </material>
-<!--BASE_LINK-->
-    <link name="base_link">
-    </link>
-<!--Base_footprint-->
-    <joint name="base_footprint_joint" type="fixed">
-        <origin xyz="0.0 0.0 0.0" rpy="0.0 0.0 0.0"/>
-        <parent link="base_link"/>
-        <child link="base_footprint"/>
-        <axis xyz="0.0 0.0 0.0"/>
-    </joint>
-    <link name="base_footprint">
-    </link>
-<!--CHASSIS_LINK-->
-    <joint name="chassis_joint" type="fixed">
-        <origin xyz="-0.1 0.0 0.0"/>
-        <parent link="base_link"/>
-        <child link="chassis_link"/>
-    </joint>
-    <link name="chassis_link">
-        <visual>
-            <origin xyz="0.15 0.0 0.04" rpy="0.0 0.0 0.0"/>
-            <geometry>
-                <box size="0.3 0.185 0.08"/>
-            </geometry>
-            <material name="gold"/>
-        </visual>
-        <collision>
-            <origin xyz="0.15 0.0 0.04" rpy="0.0 0.0 0.0"/>
-            <geometry>
-                <box size="0.3 0.185 0.08"/>
-            </geometry>
-        </collision>
-        <xacro:inertial_box mass="0.4" x="0.3" y="0.185" z="0.08">
-            <origin xyz="0.15 0 0.04" rpy=" 0 0 0"/>
-        </xacro:inertial_box>
-    </link>
-    <gazebo reference="chassis_link">
-        <material>Gazebo/Gold</material>
-    </gazebo>
-<!--LEFT_WHEEL-->
-    <joint name="left_wheel_joint" type="continuous">
-        <origin xyz="0.0 0.1125 0.0" rpy="-${pi/2} 0.0 0.0"/>
-        <parent link="base_link"/>
-        <child link="left_wheel"/>
-        <axis xyz="0.0 0.0 1.0"/>
-    </joint>
-    <link name="left_wheel">
-        <visual>
-            <geometry>
-                <cylinder radius="0.04" length="0.04"/>
-            </geometry>
-            <material name="black"/>
-        </visual>
-        <collision>
-            <geometry>
-                <cylinder radius="0.04" length="0.04"/>
-            </geometry>
-        </collision>
-        <xacro:inertial_cylinder mass="0.1" radius="0.04" length="0.04">
-             <origin xyz="0 0 0" rpy=" 0 0 0"/>
-        </xacro:inertial_cylinder>
-    </link>
-    <gazebo reference="left_wheel">
-        <material>Gazebo/Black</material>
-    </gazebo>
-<!--RIGHT_WHEEL-->
-     <joint name="right_wheel_joint" type="continuous">
-        <origin xyz="0.0 -0.1125 0.0" rpy="${pi/2} 0.0 0.0"/>
-        <parent link="base_link"/>
-        <child link="right_wheel"/>
-        <axis xyz="0.0 0.0 -1.0"/>
-    </joint>
-    <link name="right_wheel">
-        <visual>
-            <geometry>
-                <cylinder radius="0.04" length="0.04"/>
-            </geometry>
-            <material name="black"/>
-        </visual>
-        <collision>
-            <geometry>
-                <cylinder radius="0.04" length="0.04"/>
-            </geometry>
-        </collision>
-        <xacro:inertial_cylinder mass="0.1" radius="0.04" length="0.04">
-             <origin xyz="0 0 0" rpy=" 0 0 0"/>
-        </xacro:inertial_cylinder>
-    </link>
-    <gazebo reference="right_wheel">
-        <material>Gazebo/Black</material>
-    </gazebo>
-<!--CASTOR_WHEEL-->
-    <joint name="castor_wheel_joint" type="fixed">
-        <origin xyz="0.24 0.0 0.0"/>
-        <parent link="chassis_link"/>
-        <child link="castor_wheel"/>
-    </joint>
-    <link name="castor_wheel">
-        <visual>
-            <geometry>
-                <sphere radius="0.04"/>
-            </geometry>
-            <material name="red"/>
-        </visual>
-        <collision>
-             <geometry>
-                <sphere radius="0.04"/>
-            </geometry>
-        </collision>
-        <xacro:inertial_sphere mass="0.1" radius="0.04">
-            <origin xyz="0 0 0" rpy=" 0 0 0"/>
-        </xacro:inertial_sphere>
-    </link>
-    <gazebo reference="castor_wheel">
-        <material>Gazebo/Red</material>
-        <mu1 value="0.001"/>
-        <mu2 value="0.001"/>
-    </gazebo>
+    <material name="blue">
+        <color rgba="0.0 0.0 1.0 1.0"/>
+    </material>
+    <link
+    name="base_link">
+  </link>
+  <link
+    name="left_wheel">
+    <inertial>
+      <origin
+        xyz="-8.83488102121355E-10 5.46856449012978E-11 -0.00153990809638952"
+        rpy="0 0 0" />
+      <mass
+        value="0.0351743518689195" />
+      <inertia
+        ixx="1.52365643010477E-05"
+        ixy="3.0840857389948E-10"
+        ixz="-9.97409077694242E-14"
+        iyy="1.5237343017232E-05"
+        iyz="-6.11272444343794E-14"
+        izz="2.57855724460667E-05" />
+    </inertial>
+    <visual>
+      <origin
+        xyz="0 0 0"
+        rpy="0 0 0" />
+      <geometry>
+        <mesh
+          filename="package://medox_robot/meshes/left_wheel.STL" />
+      </geometry>
+      <material name="blue" />
+    </visual>
+    <collision>
+      <origin
+        xyz="0 0 0"
+        rpy="0 0 0" />
+      <geometry>
+        <mesh
+          filename="package://medox_robot/meshes/left_wheel.STL" />
+      </geometry>
+    </collision>
+  </link>
+  <joint
+    name="left_wheel_joint"
+    type="continuous">
+    <origin
+      xyz="0 0.138 -0.0210000000000002"
+      rpy="-1.5707963267949 0 0" />
+    <parent
+      link="base_link" />
+    <child
+      link="left_wheel" />
+    <axis
+      xyz="0 0 1" />
+  </joint>
+  <link
+    name="right_wheel">
+    <inertial>
+      <origin
+        xyz="7.70630951413276E-10 -3.32503330424672E-10 -0.00153990805361556"
+        rpy="0 0 0" />
+      <mass
+        value="0.0351743514548104" />
+      <inertia
+        ixx="1.52365640491052E-05"
+        ixy="3.08509166722093E-10"
+        ixz="8.38334222583704E-14"
+        iyy="1.52373429696304E-05"
+        iyz="2.27587680472107E-14"
+        izz="2.57855721584521E-05" />
+    </inertial>
+    <visual>
+      <origin
+        xyz="0 0 0"
+        rpy="0 0 0" />
+      <geometry>
+        <mesh
+          filename="package://medox_robot/meshes/right_wheel.STL" />
+      </geometry>
+      <material name="blue" />
+    </visual>
+    <collision>
+      <origin
+        xyz="0 0 0"
+        rpy="0 0 0" />
+      <geometry>
+        <mesh
+          filename="package://medox_robot/meshes/right_wheel.STL" />
+      </geometry>
+    </collision>
+  </link>
+  <joint
+    name="right_wheel_joint"
+    type="continuous">
+    <origin
+      xyz="0 -0.138 -0.0210000000000002"
+      rpy="1.5707963267949 0 0" />
+    <parent
+      link="base_link" />
+    <child
+      link="right_wheel" />
+    <axis
+      xyz="0 0 1" />
+  </joint>
+  <link
+    name="castor_wheel_f">
+    <inertial>
+      <origin
+        xyz="0 -5.55111512312578E-17 -0.0161355568158763"
+        rpy="0 0 0" />
+      <mass
+        value="0.00448472842670636" />
+      <inertia
+        ixx="7.32465415243615E-07"
+        ixy="-1.23592415742786E-22"
+        ixz="3.531673838546E-22"
+        iyy="5.9050285314133E-07"
+        iyz="-3.23587887691373E-21"
+        izz="5.39736643368085E-07" />
+    </inertial>
+    <visual>
+      <origin
+        xyz="0 0 0"
+        rpy="0 0 0" />
+      <geometry>
+        <mesh
+          filename="package://medox_robot/meshes/castor_wheel_f.STL" />
+      </geometry>
+      <material name="black" />
+    </visual>
+    <collision>
+      <origin
+        xyz="0 0 0"
+        rpy="0 0 0" />
+      <geometry>
+        <mesh
+          filename="package://medox_robot/meshes/castor_wheel_f.STL" />
+      </geometry>
+    </collision>
+  </link>
+  <joint
+    name="castor_wheel_f_joint"
+    type="fixed">
+    <origin
+      xyz="0.1875 0 0"
+      rpy="0 0 0" />
+    <parent
+      link="base_link" />
+    <child
+      link="castor_wheel_f" />
+    <axis
+      xyz="0 0 1" />
+  </joint>
+  <link
+    name="castor_wheel_f1">
+    <inertial>
+      <origin
+        xyz="0 0 -1.38777878078145E-17"
+        rpy="0 0 0" />
+      <mass
+        value="0.0215237500041331" />
+      <inertia
+        ixx="2.68174134760054E-06"
+        ixy="5.38159277687387E-39"
+        ixz="1.07427957226757E-23"
+        iyy="2.68174134760054E-06"
+        iyz="3.20819031209118E-23"
+        izz="3.97300328662299E-06" />
+    </inertial>
+    <visual>
+      <origin
+        xyz="0 0 0"
+        rpy="0 0 0" />
+      <geometry>
+        <mesh
+          filename="package://medox_robot/meshes/castor_wheel_f1.STL" />
+      </geometry>
+      <material name="white" />
+    </visual>
+    <collision>
+      <origin
+        xyz="0 0 0"
+        rpy="0 0 0" />
+      <geometry>
+        <mesh
+          filename="package://medox_robot/meshes/castor_wheel_f1.STL" />
+      </geometry>
+    </collision>
+  </link>
+  <joint
+    name="castor_wheel_f1_jont"
+    type="fixed">
+    <origin
+      xyz="0 0 -0.0356000000000001"
+      rpy="-1.5707963267949 0 0" />
+    <parent
+      link="castor_wheel_f" />
+    <child
+      link="castor_wheel_f1" />
+    <axis
+      xyz="0 1 0" />
+  </joint>
+  <link
+    name="castor_wheel_b">
+    <inertial>
+      <origin
+        xyz="0 -5.55111512312578E-17 -0.0145355568158763"
+        rpy="0 0 0" />
+      <mass
+        value="0.00448472842670636" />
+      <inertia
+        ixx="7.32465415243615E-07"
+        ixy="-6.97731693449958E-23"
+        ixz="4.00566546990044E-22"
+        iyy="5.9050285314133E-07"
+        iyz="-3.53808807516372E-21"
+        izz="5.39736643368085E-07" />
+    </inertial>
+    <visual>
+      <origin
+        xyz="0 0 0"
+        rpy="0 0 0" />
+      <geometry>
+        <mesh
+          filename="package://medox_robot/meshes/castor_wheel_b.STL" />
+      </geometry>
+      <material name="black" />
+    </visual>
+    <collision>
+      <origin
+        xyz="0 0 0"
+        rpy="0 0 0" />
+      <geometry>
+        <mesh
+          filename="package://medox_robot/meshes/castor_wheel_b.STL" />
+      </geometry>
+    </collision>
+  </link>
+  <joint
+    name="castor_wheel_b_joint"
+    type="fixed">
+    <origin
+      xyz="-0.1875 0 0"
+      rpy="0 0 0" />
+    <parent
+      link="base_link" />
+    <child
+      link="castor_wheel_b" />
+    <axis
+      xyz="0 0 1" />
+  </joint>
+  <link
+    name="castor_wheel_b1">
+    <inertial>
+      <origin
+        xyz="5.55111512312578E-17 2.77555756156289E-17 1.38777878078145E-17"
+        rpy="0 0 0" />
+      <mass
+        value="0.0215237500041331" />
+      <inertia
+        ixx="2.68174134760053E-06"
+        ixy="5.29823666801976E-39"
+        ixz="1.20662847027604E-23"
+        iyy="2.68174134760053E-06"
+        iyz="3.20819031209118E-23"
+        izz="3.97300328662299E-06" />
+    </inertial>
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
File: description/ros2_control.xacro (robot description, xacro)
@@ -28,5 +28,5 @@
                 <param name="right_wheel_name">right_wheel_joint</param>
                 <param name="loop_rate">30</param>
-                <param name="device">/dev/ttyUSB0</param>
+                <param name="device">/dev/ttyACM0</param>
                 <param name="baud_rate">57600</param>
                 <param name="timeout">1000</param>
