Commit message: slight_changes

File: description/diff_drive_controller_plugin.xacro (robot description, xacro)
@@ -7,6 +7,6 @@
             <left_joint>left_wheel_joint</left_joint>
             <right_joint>right_wheel_joint</right_joint>
-            <wheel_separation>0.225</wheel_separation>
-            <wheel_diameter>0.08</wheel_diameter>
+            <wheel_separation>0.267</wheel_separation>
+            <wheel_diameter>0.065</wheel_diameter>
             <!--limits-->
             <max_wheel_torque>200</max_wheel_torque>

File: description/robot.urdf.xacro (robot description, xacro)
@@ -2,5 +2,5 @@
 <robot xmlns:xacro="http://www.ros.org/wiki/xacro"  name="robot">
     <xacro:include filename="robot_core.xacro" />
-    <!-- <xacro:include filename="diff_drive_controller_plugin.xacro" /> -->
+    <!--<xacro:include filename="diff_drive_controller_plugin.xacro" /> -->
     <xacro:include filename="ros2_control.xacro" />
     <xacro:include filename="lidar_plugin.xacro" />

File: description/robot_core.xacro (robot description, xacro)
@@ -18,6 +18,5 @@
     name="base_link">
   </link>
-  <link
-    name="left_wheel">
+  <link name="left_wheel">
     <inertial>
       <origin
@@ -35,7 +34,5 @@
     </inertial>
     <visual>
-      <origin
-        xyz="0 0 0"
-        rpy="0 0 0" />
+      <origin xyz="0 0 0" rpy="0 0 0" />
       <geometry>
         <mesh
@@ -45,7 +42,5 @@
     </visual>
     <collision>
-      <origin
-        xyz="0 0 0"
-        rpy="0 0 0" />
+      <origin xyz="0 0 0" rpy="0 0 0" />
       <geometry>
         <mesh
@@ -54,25 +49,14 @@
     </collision>
   </link>
-  <joint
-    name="left_wheel_joint"
-    type="continuous">
-    <origin
-      xyz="0 0.138 -0.0210000000000002"
-      rpy="-1.5707963267949 0 0" />
-    <parent
-      link="base_link" />
-    <child
-      link="left_wheel" />
-    <axis
-      xyz="0 0 1" />
-  </joint>
-  <link
-    name="right_wheel">
-    <inertial>
-      <origin
-        xyz="7.70630951413276E-10 -3.32503330424672E-10 -0.00153990805361556"
-        rpy="0 0 0" />
-      <mass
-        value="0.0351743514548104" />
+  <joint  name="left_wheel_joint" type="continuous">
+    <origin xyz="0 0.138 -0.0210000000000002" rpy="-1.5707963267949 0 0" />
+    <parent link="base_link" />
+    <child  link="left_wheel" />
+    <axis xyz="0 0 1" />
+  </joint>
+  <link name="right_wheel">
+    <inertial>
+      <origin xyz="7.70630951413276E-10 -3.32503330424672E-10 -0.00153990805361556" rpy="0 0 0" />
+      <mass value="0.0351743514548104" />
       <inertia
         ixx="1.52365640491052E-05"
@@ -84,7 +68,5 @@
     </inertial>
     <visual>
-      <origin
-        xyz="0 0 0"
-        rpy="0 0 0" />
+      <origin xyz="0 0 0" rpy="0 0 0" />
       <geometry>
         <mesh
@@ -94,7 +76,5 @@
     </visual>
     <collision>
-      <origin
-        xyz="0 0 0"
-        rpy="0 0 0" />
+      <origin xyz="0 0 0" rpy="0 0 0" />
       <geometry>
         <mesh
@@ -106,22 +86,13 @@
     name="right_wheel_joint"
     type="continuous">
-    <origin
-      xyz="0 -0.138 -0.0210000000000002"
-      rpy="1.5707963267949 0 0" />
-    <parent
-      link="base_link" />
-    <child
-      link="right_wheel" />
-    <axis
-      xyz="0 0 1" />
-  </joint>
-  <link
-    name="castor_wheel_f">
-    <inertial>
-      <origin
-        xyz="0 -5.55111512312578E-17 -0.0161355568158763"
-        rpy="0 0 0" />
-      <mass
-        value="0.00448472842670636" />
+    <origin xyz="0 -0.138 -0.0210000000000002"  rpy="-1.5707963267949 0 0" />
+    <parent link="base_link" />
+    <child  link="right_wheel" />
+    <axis xyz="0 0 1" />
+  </joint>
+  <link name="castor_wheel_f">
+    <inertial>
+      <origin xyz="0 -5.55111512312578E-17 -0.0161355568158763" rpy="0 0 0" />
+      <mass value="0.00448472842670636" />
       <inertia
         ixx="7.32465415243615E-07"
@@ -133,7 +104,5 @@
     </inertial>
     <visual>
-      <origin
-        xyz="0 0 0"
-        rpy="0 0 0" />
+      <origin xyz="0 0 0" rpy="0 0 0" />
       <geometry>
         <mesh
@@ -143,7 +112,5 @@
     </visual>
     <collision>
-      <origin
-        xyz="0 0 0"
-        rpy="0 0 0" />
+      <origin xyz="0 0 0" rpy="0 0 0" />
       <geometry>
         <mesh
@@ -152,16 +119,9 @@
     </collision>
   </link>
-  <joint
-    name="castor_wheel_f_joint"
-    type="fixed">
-    <origin
-      xyz="0.1875 0 0"
-      rpy="0 0 0" />
-    <parent
-      link="base_link" />
-    <child
-      link="castor_wheel_f" />
-    <axis
-      xyz="0 0 1" />
+  <joint name="castor_wheel_f_joint" type="fixed">
+    <origin xyz="0.1875 0 0" rpy="0 0 0" />
+    <parent link="base_link" />
+    <child link="castor_wheel_f" />
+    <axis xyz="0 0 1" />
   </joint>
   <link
@@ -182,7 +142,5 @@
     </inertial>
     <visual>
-      <origin
-        xyz="0 0 0"
-        rpy="0 0 0" />
+      <origin xyz="0 0 0" rpy="0 0 0" />
       <geometry>
         <mesh
@@ -192,7 +150,5 @@
     </visual>
     <collision>
-      <origin
-        xyz="0 0 0"
-        rpy="0 0 0" />
+      <origin xyz="0 0 0" rpy="0 0 0" />
       <geometry>
         <mesh
@@ -201,23 +157,13 @@
     </collision>
   </link>
-  <joint
-    name="castor_wheel_f1_jont"
-    type="fixed">
-    <origin
-      xyz="0 0 -0.0356000000000001"
-      rpy="-1.5707963267949 0 0" />
-    <parent
-      link="castor_wheel_f" />
-    <child
-      link="castor_wheel_f1" />
-    <axis
-      xyz="0 1 0" />
-  </joint>
-  <link
-    name="castor_wheel_b">
-    <inertial>
-      <origin
-        xyz="0 -5.55111512312578E-17 -0.0145355568158763"
-        rpy="0 0 0" />
+  <joint name="castor_wheel_f1_jont" type="fixed">
+    <origin xyz="0 0 -0.0356000000000001" rpy="-1.5707963267949 0 0" />
+    <parent link="castor_wheel_f" />
+    <child link="castor_wheel_f1" />
+    <axis xyz="0 1 0" />
+  </joint>
+  <link name="castor_wheel_b">
+    <inertial>
+      <origin xyz="0 -5.55111512312578E-17 -0.0145355568158763" rpy="0 0 0" />
       <mass
         value="0.00448472842670636" />
@@ -231,7 +177,5 @@
     </inertial>
     <visual>
-      <origin
-        xyz="0 0 0"
-        rpy="0 0 0" />
+      <origin xyz="0 0 0" rpy="0 0 0" />
       <geometry>
         <mesh
@@ -241,7 +185,5 @@
     </visual>
     <collision>
-      <origin
-        xyz="0 0 0"
-        rpy="0 0 0" />
+      <origin xyz="0 0 0" rpy="0 0 0" />
       <geometry>
         <mesh
@@ -250,23 +192,13 @@
     </collision>
   </link>
-  <joint
-    name="castor_wheel_b_joint"
-    type="fixed">
-    <origin
-      xyz="-0.1875 0 0"
-      rpy="0 0 0" />
-    <parent
-      link="base_link" />
-    <child
-      link="castor_wheel_b" />
-    <axis
-      xyz="0 0 1" />
-  </joint>
-  <link
-    name="castor_wheel_b1">
-    <inertial>
-      <origin
-        xyz="5.55111512312578E-17 2.77555756156289E-17 1.38777878078145E-17"
-        rpy="0 0 0" />
+  <joint name="castor_wheel_b_joint" type="fixed">
+    <origin xyz="-0.1875 0 0" rpy="0 0 0" />
+    <parent link="base_link" />
+    <child link="castor_wheel_b" />
+    <axis xyz="0 0 1" />
+  </joint>
+  <link name="castor_wheel_b1">
+    <inertial>
+      <origin xyz="5.55111512312578E-17 2.77555756156289E-17 1.38777878078145E-17" rpy="0 0 0" />
       <mass
         value="0.0215237500041331" />
@@ -280,7 +212,5 @@
     </inertial>
     <visual>
-      <origin
-        xyz="0 0 0"
-        rpy="0 0 0" />
+      <origin xyz="0 0 0" rpy="0 0 0" />
       <geometry>
         <mesh
@@ -290,7 +220,5 @@
     </visual>
     <collision>
-      <origin
-        xyz="0 0 0"
-        rpy="0 0 0" />
+      <origin xyz="0 0 0" rpy="0 0 0" />
       <geometry>
         <mesh
@@ -299,23 +227,13 @@
     </collision>
   </link>
-  <joint
-    name="castor_wheel_b1_joint"
-    type="fixed">
-    <origin
-      xyz="0 0 -0.034"
-      rpy="-1.5707963267949 0 0" />
-    <parent
-      link="castor_wheel_b" />
-    <child
-      link="castor_wheel_b1" />
-    <axis
-      xyz="0 1 0" />
-  </joint>
-  <link
-    name="chassis">
-    <inertial>
-      <origin
-        xyz="-2.74086309204336E-16 -1.38777878078145E-17 -0.0646619925057325"
-        rpy="0 0 0" />
+  <joint name="castor_wheel_b1_joint" type="fixed">
+    <origin xyz="0 0 -0.034" rpy="-1.5707963267949 0 0" />
+    <parent link="castor_wheel_b" />
+    <child link="castor_wheel_b1" />
+    <axis xyz="0 1 0" />
+  </joint>
+  <link name="chassis">
+    <inertial>
+      <origin xyz="-2.74086309204336E-16 -1.38777878078145E-17 -0.0646619925057325" rpy="0 0 0" />
       <mass
         value="3.0292673007409" />
@@ -329,7 +247,5 @@
     </inertial>
     <visual>
-      <origin
-        xyz="0 0 0"
-        rpy="0 0 0" />
+      <origin xyz="0 0 0" rpy="0 0 0" />
       <geometry>
         <mesh
@@ -339,7 +255,5 @@
     </visual>
     <collision>
-      <origin
-        xyz="0 0 0"
-        rpy="0 0 0" />
+      <origin xyz="0 0 0" rpy="0 0 0" />
       <geometry>
         <mesh
@@ -348,23 +262,13 @@
     </collision>
   </link>
-  <joint
-    name="chassis_joint"
-    type="fixed">
-    <origin
-      xyz="0 0 0.126"
-      rpy="0 0 0" />
-    <parent
-      link="base_link" />
-    <child
-      link="chassis" />
-    <axis
-      xyz="0 0 0" />
-  </joint>
-  <link
-    name="lidar_link">
-    <inertial>
-      <origin
-        xyz="-0.00675749326271478 0.000361476187292389 -0.00738187226715975"
-        rpy="0 0 0" />
+  <joint name="chassis_joint" type="fixed">
+    <origin xyz="0 0 0.126" rpy="0 0 0" />
+    <parent link="base_link" />
+    <child link="chassis" />
+    <axis xyz="0 0 0" />
+  </joint>
+  <link name="lidar_link">
+    <inertial>
+      <origin xyz="-0.00675749326271478 0.000361476187292389 -0.00738187226715975" rpy="0 0 0" />
       <mass
         value="1.33076913637071" />
@@ -378,7 +282,5 @@
     </inertial>
     <visual>
-      <origin
-        xyz="0 0 0"
-        rpy="0 0 0" />
+      <origin xyz="0 0 0" rpy="0 0 0" />
       <geometry>
         <mesh
@@ -388,7 +290,5 @@
     </visual>
     <collision>
-      <origin
-        xyz="0 0 0"
-        rpy="0 0 0" />
+      <origin xyz="0 0 0" rpy="0 0 0" />
       <geometry>
         <mesh
@@ -397,16 +297,9 @@
     </collision>
   </link>
-  <joint
-    name="lidar_joint"
-    type="fixed">
-    <origin
-      xyz="0.0151 0.0024244 0.04265"
-      rpy="0 0 0" />
-    <parent
-      link="chassis" />
-    <child
-      link="lidar_link" />
-    <axis
-      xyz="0 0 0" />
+  <joint name="lidar_joint" type="fixed">
+    <origin xyz="0.0151 0.0024244 0.04265" rpy="0 0 0" />
+    <parent link="chassis" />
+    <child link="lidar_link" />
+    <axis xyz="0 0 0" />
   </joint>
 </robot>
