Commit message: changes_urdf

File: description/robot_core.xacro (robot description, xacro)
@@ -18,4 +18,12 @@
     name="base_link">
   </link>
+  <joint name="base_footprint_joint" type="fixed">
+        <origin xyz="0.0 0.0 0.0" rpy="0.0 0.0 0.0"/>
+        <parent link="base_link"/>
+        <child link="base_footprint"/>
+        <axis xyz="0.0 0.0 0.0"/>
+    </joint>
+    <link name="base_footprint">
+    </link>
   <link name="left_wheel">
     <inertial>
